File: SchemV2/ftc-iowa-pin-v2.kicad_pcb (KiCad board)
At the start: 2 copper layers, 37.9 x 24.3 mm, 62 parts, among them Q101 BSS84, Q102 BSS84, SW101 POWER, U101 TPS61220, U102 PIC16LF1704

Commit message: Added copper pour
Routing:
- net GND: track 77.7 -> 94.3 mm, vias 4 -> 5
- added copper zone on B.Cu, net GND
- added copper zone on F.Cu, net GND

Commit message: cleaned up silk
Routing:
- net /VSYS: track 25.9 -> 25.4 mm

Commit message: schematic
Routing:
- net GND: track 94.3 -> 196.2 mm, vias 5 -> 14
- net /SEL0_ANODE: track 35.4 -> 36.5 mm
- net N-0000037: track 21.2 -> 22.2 mm
- net /MCU_VSYS: track 28.7 -> 29.6 mm
- net N-0000023: track 17.1 -> 17.7 mm
